File: battery_charger.kicad_pcb (KiCad board)
At the start: 2 copper layers, 38.4 x 33 mm, 16 parts, among them J1 Conn_01x02_Male, J2 Conn_01x02_Male, J3 USB_B_Micro, SW1 SW_Push, U1 TP4056, U2 ATmega328P-AU, Y1 Crystal

Commit message: included dimensions
Routing:
- net Vin: vias 3 -> 2
Changed lines of the file:
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@@
   (general
     (thickness 1.6)
-    (drawings 13)
-    (tracks 286)
+    (drawings 21)
+    (tracks 285)
     (zones 0)
     (modules 16)
@@
     (descr "Through hole straight pin header, 1x02, 2.54mm pitch, single row")
     (tags "Through hole pin header THT 1x02 2.54mm single row")
-    (fp_text reference J1 (at 0 -2.33 90) (layer F.SilkS)
+    (fp_text reference J1 (at -2.413 1.397) (layer F.SilkS)
       (effects (font (size 1 1) (thickness 0.15)))
     )
@@
     (descr "Generic Phoenix Contact connector footprint for: MC_1,5/2-G-3.5; number of pins: 02; pin pitch: 3.50mm; Angled || order number: 1844210 8A 160V")
     (tags "phoenix_contact connector MC_01x02_G_3.5mm")
-    (fp_text reference J2 (at 1.75 -3) (layer F.SilkS)
+    (fp_text reference J2 (at -3.937 2.794) (layer F.SilkS)
       (effects (font (size 1 1) (thickness 0.15)))
     )
@@
     )
   )
+  (dimension 12.573 (width 0.12) (layer F.SilkS)
+    (gr_text "12.573 mm" (at 111.76 102.9335 270) (layer F.SilkS)
+      (effects (font (size 1 1) (thickness 0.15)))
+    )
+    (feature1 (pts (xy 116.586 109.22) (xy 112.443579 109.22)))
+    (feature2 (pts (xy 116.586 96.647) (xy 112.443579 96.647)))
+    (crossbar (pts (xy 113.03 96.647) (xy 113.03 109.22)))
+    (arrow1a (pts (xy 113.03 109.22) (xy 112.443579 108.093496)))
+    (arrow1b (pts (xy 113.03 109.22) (xy 113.616421 108.093496)))
+    (arrow2a (pts (xy 113.03 96.647) (xy 112.443579 97.773504)))
+    (arrow2b (pts (xy 113.03 96.647) (xy 113.616421 97.773504)))
+  )
+  (dimension 5.207 (width 0.12) (layer F.SilkS)
+    (gr_text "5.207 mm" (at 119.1895 87.63) (layer F.SilkS)
+      (effects (font (size 1 1) (thickness 0.15)))
+    )
+    (feature1 (pts (xy 116.586 96.647) (xy 116.586 88.313579)))
+    (feature2 (pts (xy 121.793 96.647) (xy 121.793 88.313579)))
+    (crossbar (pts (xy 121.793 88.9) (xy 116.586 88.9)))
+    (arrow1a (pts (xy 116.586 88.9) (xy 117.712504 88.313579)))
+    (arrow1b (pts (xy 116.586 88.9) (xy 117.712504 89.486421)))
+    (arrow2a (pts (xy 121.793 88.9) (xy 120.666496 88.313579)))
+    (arrow2b (pts (xy 121.793 88.9) (xy 120.666496 89.486421)))
+  )
+  (dimension 5.057726 (width 0.12) (layer F.SilkS)
+    (gr_text "5.058 mm" (at 119.425112 91.591091 51.11550357) (layer F.SilkS)
+      (effects (font (size 1 1) (thickness 0.15)))
+    )
+    (feature1 (pts (xy 121.666 96.647) (xy 118.36972 93.98871)))
+    (feature2 (pts (xy 124.841 92.71) (xy 121.54472 90.05171)))
+    (crossbar (pts (xy 122.001197 90.419837) (xy 118.826197 94.356837)))
+    (arrow1a (pts (xy 118.826197 94.356837) (xy 119.076885 93.111825)))
+    (arrow1b (pts (xy 118.826197 94.356837) (xy 119.98984 93.848079)))
+    (arrow2a (pts (xy 122.001197 90.419837) (xy 120.837554 90.928595)))
+    (arrow2b (pts (xy 122.001197 90.419837) (xy 121.750509 91.664849)))
+  )
+  (dimension 16.51 (width 0.12) (layer F.SilkS)
+    (gr_text "16.510 mm" (at 120.777 84.455 270) (layer F.SilkS)
+      (effects (font (size 1 1) (thickness 0.15)))
+    )
+    (feature1 (pts (xy 124.841 92.71) (xy 121.460579 92.71)))
+    (feature2 (pts (xy 124.841 76.2) (xy 121.460579 76.2)))
+    (crossbar (pts (xy 122.047 76.2) (xy 122.047 92.71)))
+    (arrow1a (pts (xy 122.047 92.71) (xy 121.460579 91.583496)))
+    (arrow1b (pts (xy 122.047 92.71) (xy 122.633421 91.583496)))
+    (arrow2a (pts (xy 122.047 76.2) (xy 121.460579 77.326504)))
+    (arrow2b (pts (xy 122.047 76.2) (xy 122.633421 77.326504)))
+  )
+  (dimension 30.099 (width 0.12) (layer F.SilkS)
+    (gr_text "30.099 mm" (at 139.8905 68.707) (layer F.SilkS)
+      (effects (font (size 1 1) (thickness 0.15)))
+    )
+    (feature1 (pts (xy 124.841 76.2) (xy 124.841 69.390579)))
+    (feature2 (pts (xy 154.94 76.2) (xy 154.94 69.390579)))
+    (crossbar (pts (xy 154.94 69.977) (xy 124.841 69.977)))
+    (arrow1a (pts (xy 124.841 69.977) (xy 125.967504 69.390579)))
+    (arrow1b (pts (xy 124.841 69.977) (xy 125.967504 70.563421)))
+    (arrow2a (pts (xy 154.94 69.977) (xy 153.813496 69.390579)))
+    (arrow2b (pts (xy 154.94 69.977) (xy 153.813496 70.563421)))
+  )
+  (dimension 33.02 (width 0.12) (layer F.SilkS)
+    (gr_text "33.020 mm" (at 158.496 92.71 270) (layer F.SilkS)
+      (effects (font (size 1 1) (thickness 0.15)))
+    )
+    (feature1 (pts (xy 154.94 109.22) (xy 157.812421 109.22)))
+    (feature2 (pts (xy 154.94 76.2) (xy 157.812421 76.2)))
+    (crossbar (pts (xy 157.226 76.2) (xy 157.226 109.22)))
+    (arrow1a (pts (xy 157.226 109.22) (xy 156.639579 108.093496)))
+    (arrow1b (pts (xy 157.226 109.22) (xy 157.812421 108.093496)))
+    (arrow2a (pts (xy 157.226 76.2) (xy 156.639579 77.326504)))
+    (arrow2b (pts (xy 157.226 76.2) (xy 157.812421 77.326504)))
+  )
+  (dimension 38.35421 (width 0.12) (layer F.SilkS)
+    (gr_text "38.354 mm" (at 135.788216 116.898797 0.1897204308) (layer F.SilkS)
+      (effects (font (size 1 1) (thickness 0.15)))
+    )
+    (feature1 (pts (xy 154.94 109.22) (xy 154.962953 116.151722)))
+    (feature2 (pts (xy 116.586 109.347) (xy 116.608953 116.278722)))
+    (crossbar (pts (xy 116.607011 115.692304) (xy 154.961011 115.565304)))
+    (arrow1a (pts (xy 154.961011 115.565304) (xy 153.836455 116.155452)))
+    (arrow1b (pts (xy 154.961011 115.565304) (xy 153.832572 114.982617)))
+    (arrow2a (pts (xy 116.607011 115.692304) (xy 117.73545 116.274991)))
+    (arrow2b (pts (xy 116.607011 115.692304) (xy 117.731567 115.102156)))
+  )
+  (gr_circle (center 139.7 91.821) (end 139.7 91.567) (layer F.SilkS) (width 0.12))
   (gr_line (start 116.586 96.647) (end 121.793 96.647) (layer Edge.Cuts) (width 0.05))
   (gr_line (start 116.586 109.22) (end 116.586 96.647) (layer Edge.Cuts) (width 0.05))
@@
   (gr_line (start 125.349 76.2) (end 124.841 76.2) (layer Edge.Cuts) (width 0.05))
   (gr_line (start 125.603 76.2) (end 125.349 76.2) (layer Edge.Cuts) (width 0.05))
-  (gr_text VBAT (at 141.732 103.378) (layer F.SilkS)
+  (gr_text VBAT (at 145.796 104.648 270) (layer F.SilkS)
     (effects (font (size 1 1) (thickness 0.15)))
   )
@@
     (effects (font (size 1 1) (thickness 0.15)))
   )
-  (gr_text GND (at 138.303 103.505) (layer F.SilkS)
+  (gr_text GND (at 134.874 104.267 90) (layer F.SilkS)
     (effects (font (size 1 1) (thickness 0.15)))
   )
@@
   (segment (start 135.128 101.346) (end 135.128 92.583) (width 0.25) (layer B.Cu) (net 1))
   (segment (start 135.128 92.583) (end 136.017 91.694) (width 0.25) (layer B.Cu) (net 1))
-  (via (at 136.017 91.694) (size 0.8) (drill 0.4) (layers F.Cu B.Cu) (net 1))
   (segment (start 146.939 88.407351) (end 146.96539 88.433741) (width 0.25) (layer B.Cu) (net 1))
   (segment (start 146.939 88.519) (end 146.939 88.407351) (width 0.25) (layer B.Cu) (net 1))
